Commit message: add offset to tool for new disc

File: snp_prbt_description/urdf/snp_prbt_demo.urdf.xacro (robot description, xacro)
@@ -19,5 +19,5 @@
   <!-- tool -->
   <xacro:snp_tool parent="${prefix}tool0">
-    <origin  xyz="0 0 0" rpy="0 0 ${5 * pi / 4.0}" />
+    <origin  xyz="0 0 0.01" rpy="0 0 ${5 * pi / 4.0}" />
   </xacro:snp_tool>
 </robot>
